File: KDT_Hierarchical_KiBot.kicad_pcb (KiCad board)
At the start: 6 copper layers, 0 parts

Commit message: modified dru / stackup and netclasses for jlcpcb 4 layers impedance controlled stackup
Other:
- copper layers 6 -> 4
Changed lines of the file:
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@@
 	(generator_version "8.0")
 	(general
-		(thickness 1.66)
+		(thickness 1.6262)
 		(legacy_teardrops yes)
 	)
@@
 		(1 "In1.Cu" power "L2 (GND)")
 		(2 "In2.Cu" signal "L3 (Sig, PWR)")
-		(3 "In3.Cu" signal "L4 (Sig, PWR)")
-		(4 "In4.Cu" power "L5 (GND)")
 		(31 "B.Cu" signal "L6 (Sig, PWR)")
 		(32 "B.Adhes" user "B.Adhesive")
@@
 			(layer "F.Cu"
 				(type "copper")
-				(thickness 0.07)
+				(thickness 0.035)
 			)
 			(layer "dielectric 1"
 				(type "prepreg")
 				(color "FR4 natural")
-				(thickness 0.18)
+				(thickness 0.2104)
 				(material "FR4_7628")
 				(epsilon_r 4.29)
@@
 			(layer "In1.Cu"
 				(type "copper")
-				(thickness 0.035)
+				(thickness 0.0152)
 			)
 			(layer "dielectric 2"
 				(type "core")
 				(color "FR4 natural")
-				(thickness 0.4)
+				(thickness 1.065)
 				(material "FR4")
 				(epsilon_r 4.6)
@@
 			(layer "In2.Cu"
 				(type "copper")
-				(thickness 0.035)
+				(thickness 0.0152)
 			)
 			(layer "dielectric 3"
 				(type "prepreg")
 				(color "FR4 natural")
-				(thickness 0.18)
-				(material "FR4_7628")
-				(epsilon_r 4.29)
-				(loss_tangent 0.02)
-			)
-			(layer "In3.Cu"
-				(type "copper")
-				(thickness 0.035)
-			)
-			(layer "dielectric 4"
-				(type "core")
-				(color "FR4 natural")
-				(thickness 0.4)
-				(material "FR4")
-				(epsilon_r 4.6)
-				(loss_tangent 0.02)
-			)
-			(layer "In4.Cu"
-				(type "copper")
-				(thickness 0.035)
-			)
-			(layer "dielectric 5"
-				(type "prepreg")
-				(color "FR4 natural")
-				(thickness 0.18)
+				(thickness 0.2104)
 				(material "FR4_7628")
 				(epsilon_r 4.29)
@@
 			(layer "B.Cu"
 				(type "copper")
-				(thickness 0.07)
+				(thickness 0.035)
 			)
 			(layer "B.Mask"
